File: acrylic_nixie_clock_1digit/acrylic_nixie_clock.sch (KiCad schematic (older format))
At the start: 18 parts, among them J1 AVR-ISP-6, SW1 SW_Push, U1 ATtiny13A-SSU, U2 TPS61041DDC

Commit message: 問題点を修正
CH304Gの電源電圧を3.3Vに
RSTにコンデンサを追加
USBのフットプリントを修正
カードコネクタの追加
Parts:
- J1: footprint Connector_IDC:IDC-Header_2x03_P2.54mm_Vertical -> acrylic_nixie_clock_1digit:ISP-6
Changed lines of the file:
@@
 F 0 "J1" V 5533 2200 50  0000 C CNN
 F 1 "AVR-ISP-6" V 5624 2200 50  0000 C CNN
-F 2 "Connector_IDC:IDC-Header_2x03_P2.54mm_Vertical" V 5750 2200 50  0001 C CNN
+F 2 "acrylic_nixie_clock_1digit:ISP-6" V 5750 2200 50  0001 C CNN
 F 3 " ~" H 4725 1600 50  0001 C CNN
 	1    6000 2150
